File: keyboard.kicad_sch (KiCad schematic)
At the start: 73 parts, among them J1 Conn01_02, J2 Conn_01x04_Pin, J3 USB_C_Receptacle_USB2.0_16P, J4 Conn_01x06_Socket, Q1 Q_PMOS_SGD, SW1 SW_Push, SW10 SW_Push, SW11 SW_Push, SW12 SW_Push, SW13 SW_Push, SW14 SW_Push, SW15 SW_Push, SW16 SW_Push, SW17 SW_Push, SW18 SW_Push, SW19 SW_Push, SW2 SW_Push, SW20 SW_Push, SW21 SW_Push, SW22 SW_Push, SW23 SW_Push, SW3 SW_Push, SW4 SW_Push, SW5 SW_Push, SW6 SW_Push, SW7 SW_Push, SW8 SW_Push, SW9 SW_Push, U1 MDBT50Q-1MV2, U2 MCP73831-2-OT, U3 IS31FL3733-TQ

Commit message: new updates
Parts:
- removed D1: LED_RGB, symbol Device:LED_RGB
- added D25, D26, D27, D28, D30, D31, D32, D33, D34, D36, D37, D38, D39, D40, D41, D42, D43, D44, D45, D46, D47, D48: LED_RGB, symbol Device:LED_RGB
Connections:
- net LED_R1: now also U3.2 (SW1), D25.4 (BA), D25.5 (GA), D25.6 (RA), D26.4 (BA), D26.5 (GA), D26.6 (RA), D27.4 (BA), D27.5 (GA), D27.6 (RA), D28.4 (BA), D28.5 (GA), D28.6 (RA)
- net LED_R2: now reaches U3.3 (SW2)
- net LED_R2: now also D30.4 (BA), D30.5 (GA), D30.6 (RA), D31.4 (BA), D31.5 (GA), D31.6 (RA), D32.4 (BA), D32.5 (GA), D32.6 (RA), D33.4 (BA), D33.5 (GA), D33.6 (RA), D34.4 (BA), D34.5 (GA), D34.6 (RA)
- net LED_R3: now reaches U3.4 (SW3)
- net LED_R3: now also D36.4 (BA), D36.5 (GA), D36.6 (RA), D37.4 (BA), D37.5 (GA), D37.6 (RA), D38.4 (BA), D38.5 (GA), D38.6 (RA), D39.4 (BA), D39.5 (GA), D39.6 (RA), D40.4 (BA), D40.5 (GA), D40.6 (RA)
- net LED_R4: now reaches U3.6 (SW4)
- net LED_R4: now also U3.7 (SW5), D41.4 (BA), D41.5 (GA), D41.6 (RA), D42.4 (BA), D42.5 (GA), D42.6 (RA), D43.4 (BA), D43.5 (GA), D43.6 (RA), D44.4 (BA), D44.5 (GA), D44.6 (RA), D45.4 (BA), D45.5 (GA), D45.6 (RA)
- net LED_R5: now reaches U3.8 (SW6)
- net LED_R5: now also D46.4 (BA), D46.5 (GA), D46.6 (RA), D47.4 (BA), D47.5 (GA), D47.6 (RA), D48.4 (BA), D48.5 (GA), D48.6 (RA)
- net B_C1 renamed CS3
- net CS3: now also D30.3 (BK), D36.3 (BK), D41.3 (BK), D46.3 (BK)
- net G_C1 renamed CS2
- net CS2: now also D30.2 (GK), D36.2 (GK), D41.2 (GK), D46.2 (GK)
- net R_C1 renamed CS1
- net CS1: now also D30.1 (RK), D36.1 (RK), D41.1 (RK), D46.1 (RK)
- new net CS10: D27.1 (RK), D33.1 (RK), D39.1 (RK), D44.1 (RK)
- new net CS11: D27.2 (GK), D33.2 (GK), D39.2 (GK), D44.2 (GK)
- new net CS12: D27.3 (BK), D33.3 (BK), D39.3 (BK), D44.3 (BK)
- new net CS13: D28.1 (RK), D34.1 (RK), D40.1 (RK), D45.1 (RK)
- new net CS14: D28.2 (GK), D34.2 (GK), D40.2 (GK), D45.2 (GK)
- new net CS15: D28.3 (BK), D34.3 (BK), D40.3 (BK), D45.3 (BK)
- new net CS4: D25.1 (RK), D31.1 (RK), D37.1 (RK), D42.1 (RK), D47.1 (RK)
- new net CS5: D25.2 (GK), D31.2 (GK), D37.2 (GK), D42.2 (GK), D47.2 (GK)
- new net CS6: D25.3 (BK), D31.3 (BK), D37.3 (BK), D42.3 (BK), D47.3 (BK)
- new net CS7: D26.1 (RK), D32.1 (RK), D38.1 (RK), D43.1 (RK), D48.1 (RK)
- new net CS8: D26.2 (GK), D32.2 (GK), D38.2 (GK), D43.2 (GK), D48.2 (GK)
- new net CS9: D26.3 (BK), D32.3 (BK), D38.3 (BK), D43.3 (BK), D48.3 (BK)
Other:
- note added: "RGB LEDs"
- moved on the sheet: C29, C30, R10, R8, R9, U3

Commit message: power fixed
Connections:
- net VDD is gone; now on net 3V3: J2.3 (Pin_3), J4.5 (Pin_5), R5.1, R6.1
- net CS1: now also U3.16 (CS1)
- net CS10: now also U3.26 (CS10)
- net CS11: now also U3.27 (CS11)
- net CS12: now also U3.28 (CS12)
- net CS13: now also U3.30 (CS13)
- net CS14: now also U3.31 (CS14)
- net CS15: now also U3.32 (CS15)
- net CS2: now also U3.17 (CS2)
- net CS3: now also U3.18 (CS3)
- net CS4: now also U3.19 (CS4)
- net CS5: now also U3.21 (CS5)
- net CS6: now also U3.22 (CS6)
- net CS7: now also U3.23 (CS7)
- net CS8: now also U3.24 (CS8)
- net CS9: now also U3.25 (CS9)
- net LED_R4: no longer U3.7 (SW5)
- net LED_R5: now also U3.7 (SW5); no longer U3.8 (SW6)
- net LED_DATA: no longer names the net of U1.9 (P0.03)
- no-connect marks 2 -> 44
Other:
- moved on the sheet: C29, C30, R10, R8, R9, U3

Commit message: battery level and RGB status added merged battery
Parts:
- removed C1, C2, C4: 4.7uF, Capacitor_SMD:C_0805_2012Metric, symbol Device:C_Small
- removed C3, C5: 1uF, Capacitor_SMD:C_0805_2012Metric, symbol Device:C_Small
- removed J2: Conn_01x04_Pin, Connector_PinHeader_2.54mm:PinHeader_1x04_P2.54mm_Vertical, symbol Connector:Conn_01x04_Pin
- removed L1: 10uH, Inductor_SMD:L_0805_2012Metric, symbol Device:L_Small
- removed Q1: Q_PMOS_SGD, Package_TO_SOT_SMD:SOT-23, symbol Device:Q_PMOS_SGD
- removed R1: 2k, Resistor_SMD:R_0805_2012Metric, symbol Device:R_Small
- removed R4: 10k, Resistor_SMD:R_0805_2012Metric, symbol Device:R_Small
- removed U1: MDBT50Q-1MV2, RF_Module:Raytac_MDBT50Q, symbol RF_Module:MDBT50Q-1MV2
- removed U2: MCP73831-2-OT, Package_TO_SOT_SMD:SOT-23-5, symbol Battery_Management:MCP73831-2-OT
- added C10, C7: 1uF, Capacitor_SMD:C_0805_2012Metric, symbol Device:C_Small
- added C11: 4.7uF, Capacitor_SMD:C_0805_2012Metric, symbol Device:C_Small
- added C6, C8, C9: 4.7uF, symbol Device:C
- added J5: Conn_01x04_Pin, Connector_PinHeader_2.54mm:PinHeader_1x04_P2.54mm_Vertical, symbol Connector:Conn_01x04_Pin
- added L2: 10uH, Inductor_SMD:L_0805_2012Metric, symbol Device:L_Small
- added R11, R12, R13: 4.7k, symbol Device:R
- added R7: 10k, symbol Device:R
- added U2: MDBT50Q-1MV2, RF_Module:Raytac_MDBT50Q, symbol RF_Module:MDBT50Q-1MV2
- added U4: BQ24074RGT, Package_DFN_QFN:VQFN-16-1EP_3x3mm_P0.5mm_EP1.6x1.6mm, symbol Battery_Management:BQ24074RGT
Connections:
- net +5V: now also C6.1, U2.32 (VBUS), U4.13 (IN), U4.6 (EN1)
- net +BATT: now also C9.1, U4.2 (BAT), U4.3 (BAT)
- net 3V3: now also C10.2, C11.1, J5.3 (Pin_3), L2.1, U2.28 (VDD)
- net Col 0: now also U2.39 (P0.15)
- net Col 1: now also U2.38 (P0.16)
- net Col 2: now also U2.41 (P0.17)
- net Col 3: now also U2.42 (P0.19)
- net Col 4: now also U2.44 (P0.20)
- net Col 5: now also U2.43 (P0.21)
- net GND: now also C10.1, C11.2, C6.2, C7.2, C8.2, C9.2, J5.4 (Pin_4), R11.2, R12.2, R13.2, R7.1, U2.1 (GND), U2.15 (GND), U2.2 (GND), U2.33 (GND), U2.55 (GND), U4.14 (TMR), U4.17 (VSS), U4.4 (~{CE}), U4.5 (EN2), U4.8 (VSS)
- net LED_SCL: now also U2.16 (P0.27)
- net LED_SDA: now also U2.19 (P0.26)
- net Row 0: now also U2.22 (P0.06)
- net Row 1: now also U2.24 (P0.08)
- net Row 2: now also U2.37 (P0.13)
- net Row 3: now also U2.36 (P0.14)
- net TRACKPAD_INT: now also U2.48 (P0.24)
- net TRACKPAD_RST: now also U2.49 (P0.25)
- net TRACKPAD_SCL: now also U2.45 (P0.23)
- net TRACKPAD_SDA: now also U2.46 (P0.22)
- net USB_D+: now also U2.35 (D+)
- net USB_D-: now also U2.34 (D-)
- net VCC_LED renamed VCC_SYS
- net VCC_SYS: now also C7.1, C8.1, U2.30 (VDDH), U4.10 (OUT), U4.11 (OUT)
- new net: R7.2, U4.1 (TS)
- new net: R11.1, U4.12 (ILIM)
- new net: R13.1, U4.15 (ITERM)
- new net: R12.1, U4.16 (ISET)
- new net: L2.2, U2.31 (DCCH)
- new net: J5.1 (Pin_1), U2.51 (SWDIO)
- new net: J5.2 (Pin_2), U2.53 (SWDCLK)
- new net BAT_CHG: U2.9 (P0.03), U4.9 (~{CHG})
Other:
- note added: "Battery Connector"

Commit message: upgraded battery to 1.0C rapid-charging
Parts:
- added C31: 10uF, symbol Device:C
- added D50: LED_RGB, symbol Device:LED_RGB
- added R1, R4: 1M, symbol Device:R
- added R14, R15, R16: 330, symbol Device:R
- added R17: 100k, symbol Device:R
- added R18: 46.4k, symbol Device:R
- added R19: 10k, symbol Device:R
- R11: value 4.7k -> 1.1k
- R12: value 4.7k -> 590
- R13: value 4.7k -> 3.0k
Connections:
- net +5V: no longer U4.6 (EN1)
- net +BATT: now also R1.1
- net 3V3: now also U4.5 (EN2), D50.4 (BA), D50.5 (GA), D50.6 (RA), R17.1, R19.2
- net BAT_CHG: now also R19.1
- net GND: now also U4.6 (EN1), C31.2, R18.2, R4.1; no longer U4.14 (TMR), U4.5 (EN2)
- net VCC_SYS: now also C31.1
- net PGOOD: now reaches U4.7 (~{PGOOD})
- net PGOOD: now also U2.58 (P1.07), R17.2
- net BAT_SENSE: now reaches U2.11 (P0.02)
- net BAT_SENSE: now also R1.2, R4.2
- net STAT_R: now reaches U2.4 (P1.11)
- net STAT_R: now also R16.2
- net STAT_G: now reaches U2.5 (P1.12)
- net STAT_G: now also R15.1
- net STAT_B: now reaches U2.6 (P1.13)
- net STAT_B: now also R14.2
- new net: R18.1, U4.14 (TMR)
- new net: D50.1 (RK), R16.1
- new net: D50.3 (BK), R14.1
- new net: D50.2 (GK), R15.2
- no-connect marks 44 -> 38
Other:
- note added: "Battery level sense"
- note added: "RGB LED Matrix"
- note added: "Status RGB LED"
- note removed: "RGB LEDs"
- moved on the sheet: C10, C11, C29, C30, C6, C7, C8, C9, J1, J5, L2, R10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
